Commit message: Changes for ROS Noetic

File: igvc_self_drive_description/urdf/gem.urdf.xacro (robot description, xacro)
@@ -32,5 +32,5 @@
       </inertial>
     </link>
-    <joint name="wheel_${name}" type="continuous" >
+    <joint name="wheel_${name}_joint" type="continuous" >
       <parent link="base_link" />
       <child link="wheel_${name}" />
@@ -66,5 +66,5 @@
       </inertial>
     </link>
-    <joint name="steer_${name}" type="revolute" >
+    <joint name="steer_${name}_joint" type="revolute" >
       <parent link="base_link" />
       <child link="steer_${name}" />
@@ -73,5 +73,5 @@
       <limit upper="0.6" lower="-0.6" effort="0.0" velocity="0.0" />
     </joint>
-    <joint name="wheel_${name}" type="continuous" >
+    <joint name="wheel_${name}_joint" type="continuous" >
       <parent link="steer_${name}" />
       <child link="wheel_${name}" />
@@ -106,5 +106,5 @@
   <xacro:front_wheel name="fl" x="${half_wheelbase}" y="${half_front_track_width}" z="0" flip="1" />
   <xacro:front_wheel name="fr" x="${half_wheelbase}" y="${-half_front_track_width}" z="0" flip="0" />
-  <joint name="base_link" type="fixed">
+  <joint name="base_link_joint" type="fixed">
     <origin xyz="${half_wheelbase} 0 ${wheel_radius}" rpy="0 0 0"/>
     <parent link="base_footprint"/>

File: igvc_self_drive_description/urdf/gem_gazebo.urdf.xacro (robot description, xacro)
@@ -11,5 +11,5 @@
       <robotNamespace>/</robotNamespace>
       <jointName>
-          steer_fl, steer_fr, wheel_fl, wheel_fr, wheel_rl, wheel_rr
+          steer_fl_joint, steer_fr_joint, wheel_fl_joint, wheel_fr_joint, wheel_rl_joint, wheel_rr_joint
       </jointName>
       <updateRate>100</updateRate>
